File: Wheel_Encoder.kicad_pcb (KiCad board)
At the start: 2 copper layers, 25.6 x 18.5 mm, 8 parts, among them J1 Conn_01x04_Pin

Commit message: final design
Parts:
- added ?: , , F.Cu at (157.5, 107.5)
- added ?: , , F.Cu at (136.2, 107.5)
- added ?: , , F.Cu at (136.2, 121.3)
- added ?: , , F.Cu at (157.5, 121.3)
Connections:
- EN1 pad 1: (no net) -> GND
- EN1 pad 2: (no net) -> GND
Routing:
- net GND: track 33.5 -> 6.11 mm, vias 2 -> 4
- added copper zone on B.Cu, net GND
- added copper zone on F.Cu, net GND
Other:
- outline, holes or cut-outs redrawn
- board text added: "5V"
- board text added: "EnA"
- board text added: "EnB"
- board text added: "GND"
- board text added: "WAFFLE Systems 2026"
