File: Wheel_Encoder.kicad_sch (KiCad schematic)
At the start: 8 parts, among them J1 Conn_01x04_Pin

Commit message: final design
Parts:
- C1, C2: value 10nF -> 0.01uF
Changed lines of the file:
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@@
 			)
 		)
-		(property "Value" "10nF"
-			(at 123.19 82.804 90)
+		(property "Value" "0.01uF"
+			(at 124.46 82.804 90)
 			(effects
 				(font
@@
 			)
 		)
-		(property "Value" "10nF"
-			(at 170.18 83.312 90)
+		(property "Value" "0.01uF"
+			(at 171.45 83.312 90)
 			(effects
 				(font
