File: PEC_Sensor.kicad_pcb (KiCad board)
At the start: 4 copper layers, 55 x 70 mm, 71 parts, among them J1 Conn_01x02_Pin, J2 Conn_01x15_Pin, J3 Conn_01x15_Pin, J4 Sensor Coil, J5 Driver Coil, J6 Encoder, Q1 SSM3K336R, U1 AP62301WU, U2 AD8221, U3 OPA820, U4 TC4420

Commit message: improved design post symposium
Parts:
- removed the ? at (150.8, 128.0)
- removed the ? at (150.8, 64.0)
- added ?: , , F.Cu at (189.4, 95.1)
- added ?: , , F.Cu at (191.9, 95.1)
- added ?: , , F.Cu at (184.3, 95.2)
- added ?: , , F.Cu at (184.2, 87.5)
- added ?: , , F.Cu at (186.8, 85.0)
- added ?: , , F.Cu at (189.3, 87.5)
- added ?: , , F.Cu at (191.8, 87.5)
- added ?: , , F.Cu at (189.4, 92.6)
- added ?: , , F.Cu at (184.2, 85.0)
- added ?: , , F.Cu at (191.8, 90.1)
- added ?: , , F.Cu at (189.3, 90.1)
- added ?: , , F.Cu at (191.8, 82.4)
- added ?: , , F.Cu at (149.0, 127.0)
- added ?: , , F.Cu at (186.8, 90.1)
- added ?: , , F.Cu at (149.0, 63.5)
- added ?: , , F.Cu at (186.8, 92.6)
- added ?: , , F.Cu at (189.3, 82.4)
- added ?: , , F.Cu at (186.8, 82.4)
- added ?: , , F.Cu at (184.3, 92.6)
- added ?: , , F.Cu at (186.8, 87.5)
- added ?: , , F.Cu at (189.3, 85.0)
- added ?: , , F.Cu at (191.9, 92.6)
- added ?: , , F.Cu at (186.8, 95.2)
- added ?: , , F.Cu at (184.2, 82.4)
- added ?: , , F.Cu at (184.2, 90.1)
- added ?: , , F.Cu at (191.8, 85.0)
- added R12: 50Ω, Resistor_SMD:R_0603_1608Metric_Pad0.98x0.95mm_HandSolder, F.Cu at (170.5, 87.6)
- added TP1: 5V, TestPoint:TestPoint_THTPad_D2.0mm_Drill1.0mm, F.Cu at (157.8, 97.0)
- added TP2: GND, TestPoint:TestPoint_THTPad_D2.0mm_Drill1.0mm, F.Cu at (161.8, 97.1)
- R5: value 1k -> 1kΩ
- R6: value 4.7k -> 10kΩ
- RG1: value 10k -> 1kΩ
- moved C13 2.93 mm to (166.1, 83.7)
- moved C14 2.93 mm to (166.1, 81.4)
- moved C9 2.93 mm to (164.9, 90.7)
- moved U3 2.93 mm to (166.0, 86.7)
- moved R3 2.84 mm to (159.2, 81.1)
- moved R4 2.84 mm to (159.3, 85.6)
- moved R7 2.84 mm to (159.3, 78.9)
- moved C10 2.84 mm to (159.3, 83.3)
- moved J4 2.00 mm to (153.0, 71.8)
- moved ? 1.60 mm to (201.0, 127.0)
- moved ? 1.35 mm to (201.0, 63.5)
Connections:
- C10 pad 2: D32 -> Net-(U3--)
- RV1 pad 1: Net-(RV1-Pad1) -> D34
- U2 pad 7: Net-(RV1-Pad1) -> D34
- U3 pad 1: D32 -> Net-(U3--)
- U3 pad 4: D32 -> Net-(U3--)
Routing:
- net D34: track 3.64 -> 20.7 mm
- net Net-(U3--): track 0.00 -> 11.2 mm
- net D32: track 17.1 -> 7.03 mm
- net Net-(RV1-Pad1): track 7.46 -> 0.00 mm
- net 5V: track 6.34 -> 12.3 mm
- net Net-(R3-Pad2): track 6.09 -> 2.21 mm
- net Net-(J4-Pin_2): track 4.01 -> 6.01 mm
- net Net-(J4-Pin_1): track 4.01 -> 6.01 mm
- net GND: vias 55 -> 60
Other:
- board size 55 x 70 mm -> 59 x 71 mm
- board text added: "WIFI Facing This Way"
