File: PEC_Sensor.kicad_sch (KiCad schematic)
At the start: 42 parts, among them J1 Conn_01x02_Pin, J2 Conn_01x15_Pin, J3 Conn_01x15_Pin, J4 Sensor Coil, J5 Driver Coil, J6 Encoder, Q1 SSM3K336R, U1 AP62301WU, U2 AD8221, U3 OPA820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

Commit message: improved design post symposium
Parts:
- added R12: 50Ω, Resistor_SMD:R_0603_1608Metric_Pad0.98x0.95mm_HandSolder, symbol Device:R_US
- added TP1: 5V, TestPoint:TestPoint_THTPad_D2.0mm_Drill1.0mm, symbol Connector:TestPoint
- added TP2: GND, TestPoint:TestPoint_THTPad_D2.0mm_Drill1.0mm, symbol Connector:TestPoint
- RG1: value 470Ω -> 1kΩ
Connections:
- net 5V: now also TP1.1
- net D32: now also R12.1; no longer C10.2, U3.1, U3.4 (-)
- net D34: now also RV1.1, U2.7
- net GND: now also TP2.1
- new net: C10.2, R12.2, U3.1, U3.4 (-)
Other:
- moved on the sheet: C8, D1, J5, Q1, U4
